File: ModuloEnergia.kicad_sch (KiCad schematic)
At the start: 19 parts, among them J1 FUENTE 220V AC, J10 VIN- Pin, J11 VOUT+ Pin, J12 VOUT- Pin, J2 FUENTE 220V AC, J3 Borner 12V 10A, J4 Borner 12V 6A, J5 Fusible 12V 10A, J6 Screw_Terminal_01x03, J7 Borner Switch IN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

Commit message: Version mandada para PCB
Parts:
- removed J6: Screw_Terminal_01x03, TerminalBlock:TerminalBlock_Xinya_XY308-2.54-3P_1x03_P2.54mm_Horizontal, symbol Connector:Screw_Terminal_01x03
- added J40: Borner Switch IN, TerminalBlock:TerminalBlock_Xinya_XY308-2.54-2P_1x02_P2.54mm_Horizontal, symbol Connector:Screw_Terminal_01x02
- D1, D2: footprint LED_THT:LED_D3.0mm -> LED_THT:LED_D5.0mm
- J5: value Fusible 12V 10A -> Borner 12V 10A
Connections:
- net REG_IN+ is gone; now on net 12V_LIN_CAP: J9.1 (Pin_1), RV1.2 (VIN+), SW1.4
- net +12V6A: now also J40.1 (Pin_1)
- net 12V_LIN_CAP: now also J40.2 (Pin_2); no longer AC_DC2.4 (+Vout), J4.1 (Pin_1)
- new net F6A_IN: AC_DC2.4 (+Vout), J4.1 (Pin_1)
Changed lines of the file:
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@@
 	)
 	(junction
+		(at 189.23 55.88)
+		(diameter 0)
+		(color 0 0 0 0)
+	)
+	(junction
 		(at 172.72 45.72)
 		(diameter 0)
@@
 	)
 	(junction
-		(at 116.84 80.01)
-		(diameter 0)
-		(color 0 0 0 0)
-	)
-	(junction
 		(at 116.84 67.31)
 		(diameter 0)
@@
 	(wire
 		(pts
-			(xy 200.66 55.88) (xy 189.23 55.88)
+			(xy 189.23 55.88) (xy 200.66 55.88)
 		)
 		(stroke
@@
 	(wire
 		(pts
-			(xy 170.18 113.03) (xy 184.15 113.03)
-		)
-		(stroke
-			(width 0)
-			(type default)
-		)
-	)
-	(wire
-		(pts
 			(xy 251.46 39.37) (xy 241.3 39.37)
 		)
@@
 	(wire
 		(pts
+			(xy 189.23 71.12) (xy 190.5 71.12)
+		)
+		(stroke
+			(width 0)
+			(type default)
+		)
+	)
+	(wire
+		(pts
 			(xy 80.01 39.37) (xy 80.01 40.64)
 		)
@@
 	(wire
 		(pts
-			(xy 116.84 80.01) (xy 120.65 80.01)
-		)
-		(stroke
-			(width 0)
-			(type default)
-		)
-	)
-	(wire
-		(pts
 			(xy 157.48 74.93) (xy 157.48 77.47)
 		)
@@
 	(wire
 		(pts
+			(xy 189.23 55.88) (xy 189.23 71.12)
+		)
+		(stroke
+			(width 0)
+			(type default)
+		)
+	)
+	(wire
+		(pts
 			(xy 36.83 106.68) (xy 36.83 110.49)
 		)
@@
 		)
 	)
-	(label "F6A_IN"
-		(at 184.15 113.03 180)
-		(effects
-			(font
-				(size 1.27 1.27)
-			)
-			(justify right bottom)
-		)
-	)
 	(label "REG_IN-"
 		(at 208.28 66.04 0)
@@
 		)
 	)
-	(hierarchical_label "5V_FUENTE"
+	(hierarchical_label "12V_LIN_CAP"
 		(shape input)
-		(at 260.35 57.15 0)
+		(at 190.5 71.12 0)
 		(effects
 			(font
@@
 		)
 	)
-	(hierarchical_label "12V_NEMA"
+	(hierarchical_label "5V_FUENTE"
 		(shape input)
-		(at 201.93 45.72 0)
+		(at 260.35 57.15 0)
 		(effects
 			(font
@@
 		)
 	)
-	(hierarchical_label "12V_LIN_CAP"
+	(hierarchical_label "12V_NEMA"
 		(shape input)
-		(at 120.65 80.01 0)
+		(at 201.93 45.72 0)
 		(effects
 			(font
@@
 			)
 		)
-		(property "Footprint" "LED_THT:LED_D3.0mm"
+		(property "Footprint" "LED_THT:LED_D5.0mm"
 			(at 36.83 102.87 0)
 			(effects
@@
 	)
 	(symbol
+		(lib_id "Connector:Screw_Terminal_01x02")
+		(at 107.95 95.25 180)
+		(unit 1)
+		(exclude_from_sim no)
+		(in_bom yes)
+		(on_board no)
+		(dnp no)
+		(property "Reference" "J5"
+			(at 107.95 86.36 0)
+			(effects
+				(font
+					(size 1.27 1.27)
+				)
+			)
+		)
+		(property "Value" "Borner 12V 10A"
+			(at 107.95 88.9 0)
+			(effects
+				(font
+					(size 1.27 1.27)
+				)
+			)
+		)
+		(property "Footprint" "TerminalBlock:TerminalBlock_Xinya_XY308-2.54-2P_1x02_P2.54mm_Horizontal"
+			(at 107.95 95.25 0)
+			(effects
+				(font
+					(size 1.27 1.27)
+				)
+				(hide yes)
+			)
+		)
+		(property "Datasheet" "~"
+			(at 107.95 95.25 0)
+			(effects
+				(font
+					(size 1.27 1.27)
+				)
+				(hide yes)
+			)
+		)
+		(property "Description" "Generic screw terminal, single row, 01x02, script generated (kicad-library-utils/schlib/autogen/connector/)"
+			(at 107.95 95.25 0)
+			(effects
+				(font
+					(size 1.27 1.27)
+				)
+				(hide yes)
+			)
+		)
+		(pin "1"
+		)
+		(pin "2"
+		)
+		(instances
+			(project "CarroTransbordador"
+				(path "/911418d1-1173-4b7a-bef0-90371fdba379/467c15ee-83d4-40af-be24-6ac2c7c7ed2f"
+					(reference "J5")
+					(unit 1)
+				)
+			)
+		)
+	)
+	(symbol
 		(lib_id "Device:R")
 		(at 36.83 93.98 0)
@@
 	)
 	(symbol
-		(lib_id "CarroTransbordador:Convertidor 220 AC a 12 DC")
-		(at 67.31 31.75 0)
+		(lib_id "Connector:Screw_Terminal_01x02")
+		(at 165.1 118.11 180)
 		(unit 1)
 		(exclude_from_sim no)
 		(in_bom yes)
-		(on_board no)
+		(on_board yes)
 		(dnp no)
 		(fields_autoplaced yes)
-		(property "Reference" "AC_DC1"
-			(at 67.31 22.86 0)
+		(property "Reference" "J40"
+			(at 165.1 109.22 0)
 			(effects
 				(font
@@
 			)
 		)
-		(property "Value" "S-120-12 Convertidor 12V 10A"
-			(at 67.31 25.4 0)
+		(property "Value" "Borner Switch IN"
+			(at 165.1 111.76 0)
 			(effects
 				(font
@@
 			)
 		)
-		(property "Footprint" ""
-			(at 67.31 39.37 0)
+		(property "Footprint" "TerminalBlock:TerminalBlock_Xinya_XY308-2.54-2P_1x02_P2.54mm_Horizontal"
+			(at 165.1 118.11 0)
 			(effects
 				(font
@@
 			)
 		)
-		(property "Datasheet" ""
-			(at 77.47 40.64 0)
+		(property "Datasheet" "~"
+			(at 165.1 118.11 0)
 			(effects
 				(font
@@
 			)
 		)
-		(property "Description" ""
-			(at 67.31 31.75 0)
+		(property "Description" "Generic screw terminal, single row, 01x02, script generated (kicad-library-utils/schlib/autogen/connector/)"
+			(at 165.1 118.11 0)
 			(effects
 				(font
@@
 		(pin "1"
 		)
-		(pin "3"
-		)
-		(pin "4"
-		)
 		(pin "2"
 		)
@@
 			(project "CarroTransbordador"
 				(path "/911418d1-1173-4b7a-bef0-90371fdba379/467c15ee-83d4-40af-be24-6ac2c7c7ed2f"
-					(reference "AC_DC1")
+					(reference "J40")
 					(unit 1)
 				)
@@
 	)
 	(symbol
-		(lib_id "Connector:Screw_Terminal_01x02")
-		(at 107.95 95.25 180)
+		(lib_id "CarroTransbordador:Convertidor 220 AC a 12 DC")
+		(at 67.31 31.75 0)
 		(unit 1)
 		(exclude_from_sim no)
@@
 		(dnp no)
 		(fields_autoplaced yes)
-		(property "Reference" "J5"
-			(at 107.95 86.36 0)
+		(property "Reference" "AC_DC1"
+			(at 67.31 22.86 0)
 			(effects
 				(font
@@
 			)
 		)
-		(property "Value" "Fusible 12V 10A"
-			(at 107.95 88.9 0)
+		(property "Value" "S-120-12 Convertidor 12V 10A"
+			(at 67.31 25.4 0)
 			(effects
 				(font
@@
 			)
 		)
-		(property "Footprint" "TerminalBlock:TerminalBlock_Xinya_XY308-2.54-2P_1x02_P2.54mm_Horizontal"
-			(at 107.95 95.25 0)
+		(property "Footprint" ""
+			(at 67.31 39.37 0)
 			(effects
 				(font
@@
 			)
 		)
-		(property "Datasheet" "~"
-			(at 107.95 95.25 0)
+		(property "Datasheet" ""
+			(at 77.47 40.64 0)
 			(effects
 				(font
@@
 			)
 		)
-		(property "Description" "Generic screw terminal, single row, 01x02, script generated (kicad-library-utils/schlib/autogen/connector/)"
-			(at 107.95 95.25 0)
+		(property "Description" ""
+			(at 67.31 31.75 0)
 			(effects
 				(font
@@
 		(pin "1"
 		)
+		(pin "3"
+		)
+		(pin "4"
+		)
 		(pin "2"
 		)
@@
 			(project "CarroTransbordador"
 				(path "/911418d1-1173-4b7a-bef0-90371fdba379/467c15ee-83d4-40af-be24-6ac2c7c7ed2f"
-					(reference "J5")
+					(reference "AC_DC1")
 					(unit 1)
 				)
@@
 	)
 	(symbol
-		(lib_id "Connector:Screw_Terminal_01x03")
-		(at 165.1 115.57 180)
-		(unit 1)
-		(exclude_from_sim no)
-		(in_bom yes)
-		(on_board yes)
-		(dnp no)
-		(fields_autoplaced yes)
-		(property "Reference" "J6"
-			(at 165.1 106.68 0)
-			(effects
-				(font
-					(size 1.27 1.27)
-				)
-			)
-		)
-		(property "Value" "Screw_Terminal_01x03"
-			(at 165.1 109.22 0)
-			(effects
-				(font
-					(size 1.27 1.27)
-				)
-			)
-		)
-		(property "Footprint" "TerminalBlock:TerminalBlock_Xinya_XY308-2.54-3P_1x03_P2.54mm_Horizontal"
-			(at 165.1 115.57 0)
-			(effects
-				(font
-					(size 1.27 1.27)
-				)
-				(hide yes)
-			)
-		)
-		(property "Datasheet" "~"
-			(at 165.1 115.57 0)
-			(effects
-				(font
-					(size 1.27 1.27)
-				)
-				(hide yes)
-			)
-		)
-		(property "Description" "Generic screw terminal, single row, 01x03, script generated (kicad-library-utils/schlib/autogen/connector/)"
-			(at 165.1 115.57 0)
-			(effects
-				(font
-					(size 1.27 1.27)
-				)
-				(hide yes)
-			)
-		)
-		(pin "3"
-		)
-		(pin "1"
-		)
-		(pin "2"
-		)
-		(instances
-			(project ""
-				(path "/911418d1-1173-4b7a-bef0-90371fdba379/467c15ee-83d4-40af-be24-6ac2c7c7ed2f"
-					(reference "J6")
-					(unit 1)
-				)
-			)
-		)
-	)
-	(symbol
 		(lib_id "Connector:Screw_Terminal_01x02")
 		(at 165.1 97.79 180)
@@
 			)
 		)
-		(property "Footprint" "LED_THT:LED_D3.0mm"
+		(property "Footprint" "LED_THT:LED_D5.0mm"
 			(at 22.86 102.87 0)
 			(effects
