File: ModuloControladores.kicad_sch (KiCad schematic)
At the start: 24 parts, among them J13 Borner ESP32, J14 Conn. Conv. HV, J15 Conn. Conv. LV, J16 Conn. ESP32, J17 Conn. LED Tr., J18 Conn. LED Empot., J19 Conn. LED Polea, J20 Conn. LED Lineal, J21 Conn. Ctrl. Tr., J22 Conn. Ctrl. Polea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

Commit message: Version mandada para PCB
Connections:
- net 5V_ARDUINO is gone; now on net 5V_FUENTE: J14.3 (Pin_3)
- net SERIAL_RX_ARD: now also LL1.7 (HV1); no longer LL1.8 (HV2)
- net SERIAL_TX_ARD: now also LL1.8 (HV2); no longer LL1.7 (HV1)

Commit message: Nuevo step y pdf
Other:
- moved on the sheet: A1, J13, J14, J15, J16, LL1, U3
